File: Hardware/Macropad/LEDs.kicad_sch (KiCad schematic)
At the start: 16 parts, among them Q1 BC847BS,115

Commit message: Added Wheel
Parts:
- removed LED12: WS2812B, XINGLIGHT XL-1515RGBC-WS2812B:XINGLIGHT XL-1515RGBC-WS2812B, symbol XINGLIGHT XL-1515RGBC-WS2812B:XINGLIGHT_XL-1515RGBC-WS2812B
- removed Q1: BC847BS,115, BC847BS:SOT65P210X110-6N, symbol BC847BS_115:BC847BS,115
- removed R1: 2.2k, Resistor_SMD:R_0402_1005Metric, symbol Device:R
- removed R3: 10k, Resistor_SMD:R_0402_1005Metric, symbol Device:R
- added IC3: SN74LV1T08DCKR, SamacSys_Parts:SOT65P210X110-5N, symbol SamacSys_Parts:SN74LV1T08DCKR
- C6: value 10nF -> 100nF; footprint Capacitor_SMD:C_0402_1005Metric -> Capacitor_SMD:C_0603_1608Metric
Connections:
- net +5V: now also C6.2, IC3.2 (B), IC3.5 (VCC); no longer C6.1
- net ALED_DI: now also IC3.1 (A)
- net DIN 1: now also IC3.4 (Y)
- net GND: now also C6.1, IC3.3 (GND); no longer C6.2
Other:
- moved on the sheet: LED1, LED10, LED11, LED2, LED3, LED4, LED5, LED6, LED7, LED8, LED9
