File: Hardware/Macropad/Macropad.kicad_sch (KiCad schematic)
At the start: 37 parts, among them IC1 TLV77333PDBVR, J2 GSB1C41110SSHR, J3 Conn_01x04_Pin, J4 103R012BB100, U2 STM32F411C_C-E_Ux, Y2 ASDDV-16.000MHZ-LR-T

Commit message: Added Wheel
Parts:
- removed C16: 4.7uF, Capacitor_SMD:C_0805_2012Metric, symbol Device:C
- removed J4: 103R012BB100, 103R012BB100:AMPHENOL_103R012BB100, symbol 103R012BB100:103R012BB100
- removed S12: Keyswitch, MX Switches:Kailh_socket_MX_optional, symbol ScottoKeebs:Placeholder_Keyswitch
- added H10, H7, H8, H9: MountingHole, MountingHole:MountingHole_2.2mm_M2, symbol Mechanical:MountingHole
Connections:
- net I2C1_SCL is gone; now on net switch 6: U2.42 (PB6)
- net I2C1_SDA is gone; now on net switch 7: U2.43 (PB7)
- net switch 3: now also U2.17 (PA7); no longer U2.39 (PB3)
- net switch 4: now also U2.29 (PA8); no longer U2.40 (PB4)
- net switch 5: now also U2.30 (PA9); no longer U2.41 (PB5)
- net switch 6: no longer U2.16 (PA6)
- net switch 7: no longer U2.17 (PA7)
- net TMC_VH: now reaches U2.12 (PA2)
- net TMC_VL: now reaches U2.13 (PA3)
- net TMC_WH: now reaches U2.14 (PA4)
- net TMC_WL: now reaches U2.15 (PA5)
- net ALED_Rotary: now reaches U2.18 (PB0)
- net SPI1_CS: now reaches U2.38 (PA15)
- net TIM2_CH1 | Rotary 1 renamed TMC_UH
- net TIM2_CH2 | Rotary 2 renamed TMC_UL
- new net SPI1_MISO: U2.40 (PB4)
- new net SPI1_MOSI: U2.41 (PB5)
- new net SPI1_SCK: U2.39 (PB3)
- new net TMC_DIAG: U2.16 (PA6)
Other:
- added sheet BLDC_Driver (BLDC_Driver.kicad_sch)
- added sheet MA702 (MA702.kicad_sch)
- note added: "Caps and Stromlimitierer und platz für spulen damit du den motor nd höhrst (direkt zu den phasen / inline)"
- moved on the sheet: S1, S2, S3
